File: uController One.kicad_pcb (KiCad board)
At the start: 2 copper layers, 100 x 50 mm, 37 parts, among them J1 Conn_01x02, J2 USB_B, J3 Conn_01x02, J4 Conn_01x04, J5 Conn_01x12, J6 Conn_01x08, U1 LM1085-5.0, U2 LP2950-3.3_TO92, U3 ATmega328P-PU, U4 MCP2221A-I/P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

Commit message: Added Gerber and drl files.
Parts:
- added J7: Conn_01x03, Connector_PinSocket_2.54mm:PinSocket_1x03_P2.54mm_Vertical, F.Cu at (103.5, 44.0)
- added R7: 1k, Resistor_THT:R_Axial_DIN0207_L6.3mm_D2.5mm_P10.16mm_Horizontal, F.Cu at (118.1, 75.6)
- moved C5 22.9 mm to (48.9, 52.1), turned to 90 degrees
- moved C4 10.2 mm to (112.4, 82.5), turned to 270 degrees
- moved D1 8.92 mm to (117.5, 85.1)
- moved R3 6.26 mm to (110.5, 47.6)
- moved C11 4.49 mm to (96.5, 50.8)
- moved F1 4.07 mm to (125.1, 80.0)
- moved U2 1.90 mm to (112.4, 79.4)
- moved H1 1.41 mm to (45.0, 45.0)
- moved H2 1.41 mm to (45.0, 85.0)
- moved H3 1.41 mm to (135.0, 45.0)
- moved H4 1.41 mm to (135.0, 85.0)
- moved C3 1.27 mm to (112.4, 70.5)
- moved R4 0.90 mm to (118.1, 44.5)
- moved C6 0.64 mm to (89.5, 50.8)
- moved U1 0.64 mm to (101.0, 86.4)
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Connections:
- net /Power Supply Unit/5V renamed +5V
- C4 pad 1: /Power Supply Unit/3.3V -> +3V3
- J4 pad 1: /Power Supply Unit/3.3V -> /Microcontroller Unit/AREF
- J4 pad 3: /Microcontroller Unit/AREF -> +3V3
- U2 pad 1: /Power Supply Unit/3.3V -> +3V3
- U4 pad 10: (no net) -> /Microcontroller Unit/USBSCL
- U4 pad 4: (no net) -> Net-(R7-Pad2)
- U4 pad 8: (no net) -> /Microcontroller Unit/USBGP3
- U4 pad 9: (no net) -> /Microcontroller Unit/USBSDA
Routing:
- net /Power Supply Unit/3.3V: track 147.9 -> 0.00 mm
- net +3V3: track 0.00 -> 85.6 mm
- net Net-(R7-Pad2): track 0.00 -> 24.0 mm
- net +5V: track 188.1 -> 209.6 mm
- net /Microcontroller Unit/USBSDA: track 0.00 -> 11.2 mm
- net /Microcontroller Unit/USBSCL: track 0.00 -> 11.2 mm
- net /Microcontroller Unit/USBGP3: track 0.00 -> 11.2 mm
- net Net-(R6-Pad1): track 14.7 -> 23.9 mm
- net Net-(D3-Pad2): track 19.1 -> 12.0 mm
- net Net-(D1-Pad2): track 12.0 -> 6.06 mm
- net /Microcontroller Unit/AREF: track 41.6 -> 35.8 mm
- net Net-(R4-Pad1): track 36.8 -> 32.9 mm
- net Net-(R3-Pad1): track 33.2 -> 29.4 mm
- net Net-(C11-Pad1): track 5.08 -> 8.51 mm
- net /Microcontroller Unit/USBD+: track 51.7 -> 52.8 mm
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Other:
- board text added: "GP3"
- board text added: "SCL"
- board text added: "SDA"
