File: uController One.sch (KiCad schematic (older format))
At the start: 10 parts, among them J1 Conn_01x02, J2 USB_B, J3 Conn_01x02, J4 Conn_01x04, J5 Conn_01x12, J6 Conn_01x08

Commit message: Added Gerber and drl files.
Parts:
- added J7: Conn_01x03, Connector_PinSocket_2.54mm:PinSocket_1x03_P2.54mm_Vertical, symbol Connector_Generic:Conn_01x03
Connections:
- net Power Supply Unit/3.3V is gone; now on net Microcontroller Unit/AREF: J4.1 (Pin_1)
- net Microcontroller Unit/AREF: no longer J4.3 (Pin_3)
- net Microcontroller Unit/VCC renamed +5V
- new net +3V3: J4.3 (Pin_3)
- new net Microcontroller Unit/USBGP3: J7.3 (Pin_3)
- new net Microcontroller Unit/USBSCL: J7.1 (Pin_1)
- new net Microcontroller Unit/USBSDA: J7.2 (Pin_2)
Changed lines of the file:
@@
 $EndDescr
 $Sheet
-S 2700 2250 1000 400
+S 2700 2250 1000 300
 U 5D4FDCE9
 F0 "Power Supply Unit" 50
 F1 "PSU.sch" 50
 F2 "VUSB" I L 2700 2450 50
-F3 "5V" I R 3700 2450 50
-F4 "3.3V" I R 3700 2350 50
-F5 "GND" I R 3700 2550 50
-F6 "VIN" I L 2700 2350 50
+F3 "VIN" I L 2700 2350 50
 $EndSheet
 $Comp
@@
 	2150 3500 2200 3500
 Wire Wire Line
-	3800 2550 3700 2550
-Wire Wire Line
-	3800 2550 3800 2650
-$Comp
-L power:GND #PWR03
-U 1 1 5D652882
-P 3800 2650
-F 0 "#PWR03" H 3800 2400 50  0001 C CNN
-F 1 "GND" H 3805 2477 50  0000 C CNN
-F 2 "" H 3800 2650 50  0001 C CNN
-F 3 "" H 3800 2650 50  0001 C CNN
-	1    3800 2650
-	1    0    0    -1
-$EndComp
-Wire Wire Line
 	4250 3000 2500 3000
 Wire Wire Line
@@
 Wire Wire Line
 	2600 2800 2500 2800
-$Comp
-L power:GND #PWR06
-U 1 1 5D650B5B
-P 5450 4850
-F 0 "#PWR06" H 5450 4600 50  0001 C CNN
-F 1 "GND" H 5455 4677 50  0000 C CNN
-F 2 "" H 5450 4850 50  0001 C CNN
-F 3 "" H 5450 4850 50  0001 C CNN
-	1    5450 4850
-	1    0    0    -1
-$EndComp
-Wire Wire Line
-	5450 4750 5450 4850
-Wire Wire Line
-	5450 4750 5350 4750
 Wire Wire Line
 	5350 2450 5850 2450
@@
 	1    0    0    -1
 $EndComp
-Wire Wire Line
-	4250 2450 3900 2450
 $Comp
 L power:GND #PWR04
@@
 	1    0    0    -1
 $EndComp
-Wire Wire Line
-	4000 1800 4250 1800
-Wire Wire Line
-	4250 1700 3900 1700
-Wire Wire Line
-	4250 1600 3800 1600
-Wire Wire Line
-	3700 2350 3800 2350
-Wire Wire Line
-	3800 1600 3800 2350
-Wire Wire Line
-	3900 1700 3900 2450
-Connection ~ 3900 2450
-Wire Wire Line
-	3900 2450 3700 2450
-Wire Wire Line
-	4000 2550 4250 2550
-Wire Wire Line
-	4000 1800 4000 2550
 $Comp
 L power:GND #PWR02
@@
 Wire Wire Line
 	5850 3550 5350 3550
-$Sheet
-S 4250 2350 1100 2500
-U 5D4FDBB8
-F0 "Microcontroller Unit" 50
-F1 "MCU.sch" 50
-F2 "VCC" I L 4250 2450 50
-F3 "GND" I R 5350 4750 50
-F4 "USBD+" I L 4250 3000 50
-F5 "USBD-" I L 4250 3100 50
-F6 "PD0" I R 5350 3750 50
-F7 "PD1" I R 5350 3850 50
-F8 "PD2" I R 5350 3950 50
-F9 "PD3" I R 5350 4050 50
-F10 "PD4" I R 5350 4150 50
-F11 "PD5" I R 5350 4250 50
-F12 "PD6" I R 5350 4350 50
-F13 "PD7" I R 5350 4450 50
-F14 "PB0" I R 5350 3550 50
-F15 "PB1" I R 5350 3450 50
-F16 "PB2" I R 5350 3350 50
-F17 "PB3" I R 5350 3250 50
-F18 "PB4" I R 5350 3150 50
-F19 "PB5" I R 5350 3050 50
-F20 "PC0" I R 5350 2950 50
-F21 "PC1" I R 5350 2850 50
-F22 "PC2" I R 5350 2750 50
-F23 "PC3" I R 5350 2650 50
-F24 "PC4" I R 5350 2550 50
-F25 "PC5" I R 5350 2450 50
-F26 "AREF" I L 4250 2550 50
-F27 "RESET" I L 4250 4650 50
-$EndSheet
 Wire Wire Line
 	2600 2250 2250 2250
@@
 	4250 1900 4150 1900
 $Comp
-L power:PWR_FLAG #FLG0101
+L power:PWR_FLAG #FLG01
 U 1 1 5DF3F549
 P 2450 1600
-F 0 "#FLG0101" H 2450 1675 50  0001 C CNN
+F 0 "#FLG01" H 2450 1675 50  0001 C CNN
 F 1 "PWR_FLAG" H 2450 1773 50  0000 C CNN
 F 2 "" H 2450 1600 50  0001 C CNN
@@
 Wire Wire Line
 	2450 2350 2700 2350
+Wire Wire Line
+	3950 1600 4250 1600
+Wire Wire Line
+	5850 4850 5350 4850
+Wire Wire Line
+	5850 4750 5350 4750
+Wire Wire Line
+	5850 4650 5350 4650
+$Comp
+L Connector_Generic:Conn_01x03 J7
+U 1 1 5DFD3048
+P 6050 4750
+F 0 "J7" H 6130 4792 50  0000 L CNN
+F 1 "Conn_01x03" H 6130 4701 50  0000 L CNN
+F 2 "Connector_PinSocket_2.54mm:PinSocket_1x03_P2.54mm_Vertical" H 6050 4750 50  0001 C CNN
+F 3 "~" H 6050 4750 50  0001 C CNN
+	1    6050 4750
+	1    0    0    -1
+$EndComp
+$Sheet
+S 4250 2350 1100 2600
+U 5D4FDBB8
+F0 "Microcontroller Unit" 50
+F1 "MCU.sch" 50
+F2 "USBD+" I L 4250 3000 50
+F3 "USBD-" I L 4250 3100 50
+F4 "PD0" I R 5350 3750 50
+F5 "PD1" I R 5350 3850 50
+F6 "PD2" I R 5350 3950 50
+F7 "PD3" I R 5350 4050 50
+F8 "PD4" I R 5350 4150 50
+F9 "PD5" I R 5350 4250 50
+F10 "PD6" I R 5350 4350 50
+F11 "PD7" I R 5350 4450 50
+F12 "PB0" I R 5350 3550 50
+F13 "PB1" I R 5350 3450 50
+F14 "PB2" I R 5350 3350 50
+F15 "PB3" I R 5350 3250 50
+F16 "PB4" I R 5350 3150 50
+F17 "PB5" I R 5350 3050 50
+F18 "PC0" I R 5350 2950 50
+F19 "PC1" I R 5350 2850 50
+F20 "PC2" I R 5350 2750 50
+F21 "PC3" I R 5350 2650 50
+F22 "PC4" I R 5350 2550 50
+F23 "PC5" I R 5350 2450 50
+F24 "AREF" I L 4250 2450 50
+F25 "RESET" I L 4250 4650 50
+F26 "USBGP3" I R 5350 4850 50
+F27 "USBSCL" I R 5350 4650 50
+F28 "USBSDA" I R 5350 4750 50
+$EndSheet
+$Comp
+L power:+5V #PWR?
+U 1 1 5E02F316
+P 3800 1600
+F 0 "#PWR?" H 3800 1450 50  0001 C CNN
+F 1 "+5V" H 3815 1773 50  0000 C CNN
+F 2 "" H 3800 1600 50  0001 C CNN
+F 3 "" H 3800 1600 50  0001 C CNN
+	1    3800 1600
+	1    0    0    -1
+$EndComp
+$Comp
+L power:+3.3V #PWR?
+U 1 1 5E038F6D
+P 3550 1600
+F 0 "#PWR?" H 3550 1450 50  0001 C CNN
+F 1 "+3.3V" H 3565 1773 50  0000 C CNN
+F 2 "" H 3550 1600 50  0001 C CNN
+F 3 "" H 3550 1600 50  0001 C CNN
+	1    3550 1600
+	1    0    0    -1
+$EndComp
+Wire Wire Line
+	4250 1700 3800 1700
+Wire Wire Line
+	3800 1700 3800 1600
+Wire Wire Line
+	4250 1800 3550 1800
+Wire Wire Line
+	3550 1800 3550 1600
+Wire Wire Line
+	4250 2450 3950 2450
+Wire Wire Line
+	3950 2450 3950 1600
 $EndSCHEMATC
